File: KiCad/Le Chiffre v2/LeChiffre.kicad_sch (KiCad schematic)
At the start: 135 parts, among them J2 Conn_01x04_Female, Q1 AO3401A, Q2 AO3400A, SW1 SW_Push, SW10 SW_Push, SW11 SW_Push, SW12 SW_Push, SW13 SW_Push, SW14 SW_Push, SW15 SW_Push, SW16 SW_Push, SW17 SW_Push, SW18 SW_Push, SW19 SW_Push, SW2 SW_Push, SW20 SW_Push, SW21 SW_Push, SW22 SW_Push, SW23 SW_Push, SW24 SW_Push, SW25 SW_Push, SW26 SW_Push, SW27 SW_Push, SW28 SW_Push, SW29 SW_Push, SW3 SW_Push, SW30 SW_Push, SW31 SW_Push, SW32 SW_Push, SW33 SW_Push, SW34 SW_Push, SW35 SW_Push, SW36 Rotary_Encoder_Switch, SW37 SW_Push, SW38 SW_Push, SW39 SW_Push, SW4 SW_Push, SW5 SW_Push, SW6 SW_Push, SW7 SW_Push, SW8 SW_Push, SW9 SW_Push, U1 elite-nano-combo-controller, U2 SN74HC595

Commit message: bom's long delayed forehead
Parts:
- added D85, D86: 1N4001, Diode_THT:D_DO-41_SOD81_P10.16mm_Horizontal, symbol Diode:1N4001
- added J1: Barrel_Jack, Connector_BarrelJack:BarrelJack_Wuerth_6941xx301002, symbol Connector:Barrel_Jack
- added K1: DIPxx-1Axx-11x, Relay_THT:Relay_StandexMeder_DIP_LowProfile, symbol Relay:DIPxx-1Axx-11x
- added L1: ElectromagneticActor, Connector_JST:JST_PH_B2B-PH-K_1x02_P2.00mm_Vertical, symbol Device:ElectromagneticActor
- added Q3: TIP120, Package_TO_SOT_THT:TO-220-3_Vertical, symbol Transistor_BJT:TIP120
Connections:
- net GND: now also Q3.3 (E)
- net VCC: now also D85.1 (K), K1.6
- net solenoid: now reaches U1.9 (6/PD7)
- net solenoid: now also Q3.1 (B)
- new net: J1.1, K1.7, K1.8
- new net: D86.2 (A), J1.2, L1.1 (-)
- new net: D86.1 (K), K1.1, K1.14, L1.2 (+)
- new net: D85.2 (A), K1.2, Q3.2 (C)
- no-connect marks 10 -> 9
