File: KiCad/Le Chiffre v2/LeChiffre.kicad_pcb (KiCad board)
At the start: 2 copper layers, 228.4 x 95.7 mm, 134 parts, among them J1 Conn_01x06_Socket, J2 Conn_01x04_Female, SW1 SW_Push, SW10 SW_Push, SW11 SW_Push, SW12 SW_Push, SW13 SW_Push, SW14 SW_Push, SW15 SW_Push, SW16 SW_Push, SW17 SW_Push, SW18 SW_Push, SW19 SW_Push, SW2 SW_Push, SW20 SW_Push, SW21 SW_Push, SW22 SW_Push, SW23 SW_Push, SW24 SW_Push, SW25 SW_Push, SW26 SW_Push, SW27 SW_Push, SW28 SW_Push, SW29 SW_Push, SW3 SW_Push, SW30 SW_Push, SW31 SW_Push, SW32 SW_Push, SW33 SW_Push, SW34 SW_Push, SW35 SW_Push, SW36 Rotary_Encoder_Switch, SW37 SW_Push, SW38 SW_Push, SW39 SW_Push, SW4 SW_Push, SW5 SW_Push, SW6 SW_Push, SW7 SW_Push, SW8 SW_Push, SW9 SW_Push, U1 pro-micro-controller, U2 SN74HC595

Commit message: fixed diode orientation to work with shift register
Parts:
- turned D1 to -90 degrees
- turned D10 to -90 degrees
- turned D11 to -90 degrees
- turned D12 to -90 degrees
- turned D13 to -90 degrees
- turned D14 to -90 degrees
- turned D15 to -90 degrees
- turned D16 to -90 degrees
- turned D17 to -90 degrees
- turned D18 to -90 degrees
- turned D19 to -90 degrees
- turned D2 to -90 degrees
- turned D20 to -90 degrees
- turned D21 to -90 degrees
- turned D22 to -90 degrees
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Connections:
- D1 pad 1: Net-(D1-K) -> row0
- D1 pad 2: row0 -> Net-(D1-A)
- D10 pad 1: Net-(D10-K) -> row0
- D10 pad 2: row0 -> Net-(D10-A)
- D11 pad 1: Net-(D11-K) -> row1
- D11 pad 2: row1 -> Net-(D11-A)
- D12 pad 1: Net-(D12-K) -> row2
- D12 pad 2: row2 -> Net-(D12-A)
- D13 pad 1: Net-(D13-K) -> row4
- D13 pad 2: row4 -> Net-(D13-A)
- D14 pad 1: Net-(D14-K) -> row0
- D14 pad 2: row0 -> Net-(D14-A)
- D15 pad 1: Net-(D15-K) -> row1
- D15 pad 2: row1 -> Net-(D15-A)
- D16 pad 1: Net-(D16-K) -> row2
- D16 pad 2: row2 -> Net-(D16-A)
- D17 pad 1: Net-(D17-K) -> row4
- D17 pad 2: row4 -> Net-(D17-A)
- D18 pad 1: Net-(D18-K) -> row0
- D18 pad 2: row0 -> Net-(D18-A)
- D19 pad 1: Net-(D19-K) -> row1
- D19 pad 2: row1 -> Net-(D19-A)
- D2 pad 1: Net-(D2-K) -> row1
- D2 pad 2: row1 -> Net-(D2-A)
- D20 pad 1: Net-(D20-K) -> row2
- D20 pad 2: row2 -> Net-(D20-A)
- D21 pad 1: Net-(D21-K) -> row4
- D21 pad 2: row4 -> Net-(D21-A)
- D22 pad 1: Net-(D22-K) -> row0
- D22 pad 2: row0 -> Net-(D22-A)
- D23 pad 1: Net-(D23-K) -> row1
- D23 pad 2: row1 -> Net-(D23-A)
- D24 pad 1: Net-(D24-K) -> row2
- D24 pad 2: row2 -> Net-(D24-A)
- D25 pad 1: Net-(D25-K) -> row4
- D25 pad 2: row4 -> Net-(D25-A)
- D26 pad 1: Net-(D26-K) -> row0
- D26 pad 2: row0 -> Net-(D26-A)
- D27 pad 1: Net-(D27-K) -> row1
- D27 pad 2: row1 -> Net-(D27-A)
- D28 pad 1: Net-(D28-K) -> row2
- D28 pad 2: row2 -> Net-(D28-A)
- D29 pad 1: Net-(D29-K) -> row3
- D29 pad 2: row3 -> Net-(D29-A)
- D3 pad 1: Net-(D3-K) -> row2
- D3 pad 2: row2 -> Net-(D3-A)
- D30 pad 1: Net-(D30-K) -> row3
- D30 pad 2: row3 -> Net-(D30-A)
- D31 pad 1: Net-(D31-K) -> row3
- D31 pad 2: row3 -> Net-(D31-A)
- D32 pad 1: Net-(D32-K) -> row3
- D32 pad 2: row3 -> Net-(D32-A)
- D33 pad 1: Net-(D33-K) -> row3
- D33 pad 2: row3 -> Net-(D33-A)
- D34 pad 1: Net-(D34-K) -> row3
- D34 pad 2: row3 -> Net-(D34-A)
- D35 pad 1: Net-(D35-K) -> row4
- D35 pad 2: row4 -> Net-(D35-A)
- D36 pad 1: Net-(D36-K) -> row4
- D36 pad 2: row4 -> Net-(D36-A)
- D37 pad 1: Net-(D37-K) -> row4
- D37 pad 2: row4 -> Net-(D37-A)
- D4 pad 1: Net-(D4-K) -> row0
- D4 pad 2: row0 -> Net-(D4-A)
- D5 pad 1: Net-(D5-K) -> row1
- D5 pad 2: row1 -> Net-(D5-A)
- D6 pad 1: Net-(D6-K) -> row2
- D6 pad 2: row2 -> Net-(D6-A)
- D7 pad 1: Net-(D7-K) -> row0
- D7 pad 2: row0 -> Net-(D7-A)
- D8 pad 1: Net-(D8-K) -> row1
- D8 pad 2: row1 -> Net-(D8-A)
- D9 pad 1: Net-(D9-K) -> row2
- D9 pad 2: row2 -> Net-(D9-A)
- SW10 pad 1: Net-(D9-K) -> Net-(D9-A)
- SW11 pad 1: Net-(D10-K) -> Net-(D10-A)
- SW12 pad 1: Net-(D11-K) -> Net-(D11-A)
- SW13 pad 1: Net-(D12-K) -> Net-(D12-A)
- SW14 pad 1: Net-(D13-K) -> Net-(D13-A)
- SW15 pad 1: Net-(D14-K) -> Net-(D14-A)
- SW16 pad 1: Net-(D15-K) -> Net-(D15-A)
- SW17 pad 1: Net-(D16-K) -> Net-(D16-A)
- SW18 pad 1: Net-(D17-K) -> Net-(D17-A)
- SW19 pad 1: Net-(D18-K) -> Net-(D18-A)
- SW2 pad 1: Net-(D1-K) -> Net-(D1-A)
- SW20 pad 1: Net-(D19-K) -> Net-(D19-A)
- SW21 pad 1: Net-(D20-K) -> Net-(D20-A)
- SW22 pad 1: Net-(D21-K) -> Net-(D21-A)
- SW23 pad 1: Net-(D22-K) -> Net-(D22-A)
- SW24 pad 1: Net-(D23-K) -> Net-(D23-A)
- SW25 pad 1: Net-(D24-K) -> Net-(D24-A)
- SW26 pad 1: Net-(D25-K) -> Net-(D25-A)
- SW27 pad 1: Net-(D26-K) -> Net-(D26-A)
- SW28 pad 1: Net-(D27-K) -> Net-(D27-A)
- SW29 pad 1: Net-(D28-K) -> Net-(D28-A)
- SW3 pad 1: Net-(D2-K) -> Net-(D2-A)
- SW30 pad 1: Net-(D29-K) -> Net-(D29-A)
- SW31 pad 1: Net-(D30-K) -> Net-(D30-A)
- SW32 pad 1: Net-(D31-K) -> Net-(D31-A)
- SW33 pad 1: Net-(D32-K) -> Net-(D32-A)
- SW34 pad 1: Net-(D33-K) -> Net-(D33-A)
- SW35 pad 1: Net-(D34-K) -> Net-(D34-A)
- SW36 pad S1: Net-(D35-K) -> Net-(D35-A)
- SW37 pad 1: Net-(D35-K) -> Net-(D35-A)
- SW38 pad 1: Net-(D36-K) -> Net-(D36-A)
- SW39 pad 1: Net-(D37-K) -> Net-(D37-A)
- SW4 pad 1: Net-(D3-K) -> Net-(D3-A)
- SW5 pad 1: Net-(D4-K) -> Net-(D4-A)
- SW6 pad 1: Net-(D5-K) -> Net-(D5-A)
- SW7 pad 1: Net-(D6-K) -> Net-(D6-A)
- SW8 pad 1: Net-(D7-K) -> Net-(D7-A)
- SW9 pad 1: Net-(D8-K) -> Net-(D8-A)
Routing:
- net Net-(D6-K): track 18.3 -> 0.00 mm
- net Net-(D6-A): track 0.00 -> 18.3 mm
- net Net-(D35-K): track 18.1 -> 0.00 mm
- net Net-(D35-A): track 0.00 -> 18.1 mm
- net Net-(D1-K): track 18.0 -> 0.00 mm
- net Net-(D1-A): track 0.00 -> 18.0 mm
- net Net-(D4-K): track 17.9 -> 0.00 mm
- net Net-(D4-A): track 0.00 -> 17.9 mm
- net Net-(D5-K): track 17.8 -> 0.00 mm
- net Net-(D5-A): track 0.00 -> 17.8 mm
- net Net-(D3-K): track 17.7 -> 0.00 mm
- net Net-(D3-A): track 0.00 -> 17.7 mm
- net Net-(D17-K): track 17.7 -> 0.00 mm
- net Net-(D17-A): track 0.00 -> 17.7 mm
- net Net-(D21-K): track 17.5 -> 0.00 mm
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